Commit message: Atlas setting updated

File: data/urdf/BioloidGP/BioloidGP.URDF (robot description, URDF)
Before this commit: robot BioloidGP, 17 links, 16 joints
Joints:
- joint l_arm: limit lower=-2.1000 upper=2.1000 effort=200 velocity=12 -> lower=-2.6180 upper=2.6180 effort=0.75 velocity=12
- joint l_foot: limit lower=-2.1000 upper=2.1000 effort=200 velocity=12 -> lower=-2.6180 upper=2.6180 effort=0.75 velocity=12
- joint l_hand: limit lower=-2.1000 upper=2.1000 effort=200 velocity=12 -> lower=-2.6180 upper=2.6180 effort=0.75 velocity=12
- joint l_heel: limit lower=-2.1000 upper=2.1000 effort=200 velocity=12 -> lower=-2.6180 upper=2.6180 effort=0.75 velocity=12
- joint l_hip: limit lower=-2.1000 upper=2.1000 effort=200 velocity=12 -> lower=-2.6180 upper=2.6180 effort=0.75 velocity=12
- joint l_shin: limit lower=-2.1000 upper=2.1000 effort=200 velocity=12 -> lower=-2.6180 upper=2.6180 effort=0.75 velocity=12
- joint l_shoulder: limit lower=-2.1000 upper=2.1000 effort=200 velocity=12 -> lower=-2.6180 upper=2.6180 effort=0.75 velocity=12
- joint l_thigh: limit lower=-2.1000 upper=2.1000 effort=200 velocity=12 -> lower=-2.6180 upper=2.6180 effort=0.75 velocity=12
- joint r_arm: limit lower=-2.1000 upper=2.1000 effort=200 velocity=12 -> lower=-2.6180 upper=2.6180 effort=0.75 velocity=12
- joint r_foot: limit lower=-2.1000 upper=2.1000 effort=200 velocity=12 -> lower=-2.6180 upper=2.6180 effort=0.75 velocity=12
- joint r_hand: limit lower=-2.1000 upper=2.1000 effort=200 velocity=12 -> lower=-2.6180 upper=2.6180 effort=0.75 velocity=12
- joint r_heel: limit lower=-2.1000 upper=2.1000 effort=200 velocity=12 -> lower=-2.6180 upper=2.6180 effort=0.75 velocity=12
- joint r_hip: limit lower=-2.1000 upper=2.1000 effort=200 velocity=12 -> lower=-2.6180 upper=2.6180 effort=0.75 velocity=12
- joint r_shin: limit lower=-2.1000 upper=2.1000 effort=200 velocity=12 -> lower=-2.6180 upper=2.6180 effort=0.75 velocity=12
- joint r_shoulder: limit lower=-2.1000 upper=2.1000 effort=200 velocity=12 -> lower=-2.6180 upper=2.6180 effort=0.75 velocity=12
- joint r_thigh: limit lower=-2.1000 upper=2.1000 effort=200 velocity=12 -> lower=-2.6180 upper=2.6180 effort=0.75 velocity=12

Commit message: Reconfigure the torque limits

File: data/urdf/BioloidGP/BioloidGP.URDF (robot description, URDF)
Before this commit: robot BioloidGP, 17 links, 16 joints
Joints:
- joint l_arm: limit lower=-2.6180 upper=2.6180 effort=0.75 velocity=12 -> lower=-2.6180 upper=2.6180 effort=1.50 velocity=12
- joint l_foot: limit lower=-2.6180 upper=2.6180 effort=0.75 velocity=12 -> lower=-2.6180 upper=2.6180 effort=1.50 velocity=12
- joint l_hand: limit lower=-2.6180 upper=2.6180 effort=0.75 velocity=12 -> lower=-2.6180 upper=2.6180 effort=1.50 velocity=12
- joint l_heel: limit lower=-2.6180 upper=2.6180 effort=0.75 velocity=12 -> lower=-2.6180 upper=2.6180 effort=1.50 velocity=12
- joint l_hip: limit lower=-2.6180 upper=2.6180 effort=0.75 velocity=12 -> lower=-2.6180 upper=2.6180 effort=1.50 velocity=12
- joint l_shin: limit lower=-2.6180 upper=2.6180 effort=0.75 velocity=12 -> lower=-2.6180 upper=2.6180 effort=1.50 velocity=12
- joint l_shoulder: limit lower=-2.6180 upper=2.6180 effort=0.75 velocity=12 -> lower=-2.6180 upper=2.6180 effort=1.50 velocity=12
- joint l_thigh: limit lower=-2.6180 upper=2.6180 effort=0.75 velocity=12 -> lower=-2.6180 upper=2.6180 effort=1.50 velocity=12
- joint r_arm: limit lower=-2.6180 upper=2.6180 effort=0.75 velocity=12 -> lower=-2.6180 upper=2.6180 effort=1.50 velocity=12
- joint r_foot: limit lower=-2.6180 upper=2.6180 effort=0.75 velocity=12 -> lower=-2.6180 upper=2.6180 effort=1.50 velocity=12
- joint r_hand: limit lower=-2.6180 upper=2.6180 effort=0.75 velocity=12 -> lower=-2.6180 upper=2.6180 effort=1.50 velocity=12
- joint r_heel: limit lower=-2.6180 upper=2.6180 effort=0.75 velocity=12 -> lower=-2.6180 upper=2.6180 effort=1.50 velocity=12
- joint r_hip: limit lower=-2.6180 upper=2.6180 effort=0.75 velocity=12 -> lower=-2.6180 upper=2.6180 effort=1.50 velocity=12
- joint r_shin: limit lower=-2.6180 upper=2.6180 effort=0.75 velocity=12 -> lower=-2.6180 upper=2.6180 effort=1.50 velocity=12
- joint r_shoulder: limit lower=-2.6180 upper=2.6180 effort=0.75 velocity=12 -> lower=-2.6180 upper=2.6180 effort=1.50 velocity=12
- joint r_thigh: limit lower=-2.6180 upper=2.6180 effort=0.75 velocity=12 -> lower=-2.6180 upper=2.6180 effort=1.50 velocity=12
